File: pcb/cubecast.kicad_pcb (KiCad board)
At the start: 2 copper layers, 1 part

Commit message: PCB started
Parts:
- removed REF**: ESP-07v2, ESP8266:ESP-07v2
- added C1: 1.0uF, Capacitors_SMD:C_0402, F.Cu at (51.6, 46.5)
- added C2: 1.0uF, Capacitors_SMD:C_0402, F.Cu at (50.2, 37.2)
- added C3: 2.2uF, Capacitors_SMD:C_0402, F.Cu at (62.2, 41.8)
- added C4: 2.2uF, Capacitors_SMD:C_0402, F.Cu at (61.8, 37.3)
- added C5: 10uF, Capacitors_SMD:C_0603_HandSoldering, F.Cu at (54.6, 40.5)
- added C6: 10uF, Capacitors_SMD:C_0603_HandSoldering, F.Cu at (55.2, 36.6)
- added C7: 0.1uF, Capacitors_SMD:C_0402, F.Cu at (48.1, 40.3)
- added C8: 0.1uF, Capacitors_SMD:C_0402, F.Cu at (45.1, 37.2)
- added OLED1: OLED_0.66_inch_64x48, OLED:OLED_0.66_inch_64x48, F.Cu at (35.6, 29.2)
- added R1: 390k, Resistors_SMD:R_0402, F.Cu at (57.8, 47.1)
- added U3: ESP-07v2, ESP8266:ESP-07v2, F.Cu at (71.9, 35.1)

Commit message: initial placement
Parts:
- U3: moved to B.Cu
- moved U3 34.8 mm to (38.1, 26.8), turned to 270 degrees
- moved C1 21.1 mm to (35.7, 32.6), turned to 270 degrees
- moved R1 17.5 mm to (49.3, 31.9)
- moved C2 13.6 mm to (37.3, 32.6), turned to 270 degrees
- moved C3 12.1 mm to (55.6, 31.6)
- moved C7 11.1 mm to (40.0, 32.6), turned to 270 degrees
- moved C4 5.38 mm to (60.1, 32.3)
- moved C8 4.98 mm to (43.4, 32.5)

Commit message: footprint for charger
Parts:
- added C10: 0.1uF, Capacitors_SMD:C_0402, F.Cu at (22.9, 37.7)
- added C9: 0.1uF, Capacitors_SMD:C_0402, F.Cu at (29.6, 37.0)
- added U1: bq24040, SMD:R-PWSON-N10, F.Cu at (26.9, 30.7)
- added U2: tps62200, TO_SOT_Packages_SMD:SOT-23-5, F.Cu at (29.1, 41.9)
Connections:
- C5 pad 1: (no net) -> /VOUT
- U3 pad 9: (no net) -> GND
Changed lines of the file:
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@@
 (kicad_pcb (version 4) (host pcbnew "(2015-08-08 BZR 6073)-product")
   (general
-    (links 22)
-    (no_connects 22)
-    (area 34.776999 26.135 88.357001 51.277001)
+    (links 32)
+    (no_connects 32)
+    (area 0 0 0 0)
     (thickness 1.6)
     (drawings 0)
     (tracks 0)
     (zones 0)
-    (modules 11)
-    (nets 10)
+    (modules 15)
+    (nets 11)
   )
   (page A4)
@@
     (36 B.SilkS user)
     (37 F.SilkS user)
-    (38 B.Mask user)
-    (39 F.Mask user)
-    (40 Dwgs.User user)
-    (41 Cmts.User user)
-    (42 Eco1.User user)
+    (38 B.Mask user hide)
+    (39 F.Mask user hide)
+    (40 Dwgs.User user hide)
+    (41 Cmts.User user hide)
+    (42 Eco1.User user hide)
     (43 Eco2.User user hide)
     (44 Edge.Cuts user hide)
     (45 Margin user)
     (46 B.CrtYd user hide)
-    (47 F.CrtYd user)
-    (48 B.Fab user)
+    (47 F.CrtYd user hide)
+    (48 B.Fab user hide)
     (49 F.Fab user hide)
   )
@@
     (pad_to_mask_clearance 0.2)
     (aux_axis_origin 0 0)
-    (visible_elements FFFFFF7F)
+    (visible_elements FFFEFF6F)
     (pcbplotparams
       (layerselection 0x00030_80000001)
@@
   (net 8 +3V3)
   (net 9 "Net-(OLED1-Pad24)")
+  (net 10 /VOUT)
   (net_class Default "This is the default net class."
     (clearance 0.2)
@@
     (uvia_drill 0.1)
     (add_net +3V3)
+    (add_net /VOUT)
     (add_net GND)
     (add_net "Net-(C1-Pad1)")
@@
     (fp_line (start -0.35 -0.6) (end 0.35 -0.6) (layer F.SilkS) (width 0.15))
     (fp_line (start 0.35 0.6) (end -0.35 0.6) (layer F.SilkS) (width 0.15))
-    (pad 1 smd rect (at -0.95 0) (size 1.2 0.75) (layers F.Cu F.Paste F.Mask))
+    (pad 1 smd rect (at -0.95 0) (size 1.2 0.75) (layers F.Cu F.Paste F.Mask)
+      (net 10 /VOUT))
     (pad 2 smd rect (at 0.95 0) (size 1.2 0.75) (layers F.Cu F.Paste F.Mask)
       (net 6 GND))
@@
     (pad 8 thru_hole oval (at 0 -14 270) (size 2.5 1.1) (drill 0.65 (offset -0.7 0)) (layers *.Cu *.Mask B.SilkS)
       (net 8 +3V3))
-    (pad 9 thru_hole oval (at 14 -14 270) (size 2.5 1.1) (drill 0.65 (offset 0.7 0)) (layers *.Cu *.Mask B.SilkS))
+    (pad 9 thru_hole oval (at 14 -14 270) (size 2.5 1.1) (drill 0.65 (offset 0.7 0)) (layers *.Cu *.Mask B.SilkS)
+      (net 6 GND))
     (pad 10 thru_hole oval (at 14 -12 270) (size 2.5 1.1) (drill 0.65 (offset 0.6 0)) (layers *.Cu *.Mask B.SilkS))
     (pad 11 thru_hole oval (at 14 -10 270) (size 2.5 1.1) (drill 0.65 (offset 0.7 0)) (layers *.Cu *.Mask B.SilkS))
@@
       (rotate (xyz 0 0 0))
     )
+  )
+  (module Capacitors_SMD:C_0402 (layer F.Cu)
+    (at 29.591 36.957)
+    (descr "Capacitor SMD 0402, reflow soldering, AVX (see smccp.pdf)")
+    (tags "capacitor 0402")
+    (attr smd)
+    (fp_text reference C9 (at 0 -1.7) (layer F.SilkS)
+      (effects (font (size 1 1) (thickness 0.15)))
+    )
+    (fp_text value 0.1uF (at 0 1.7) (layer F.Fab)
+      (effects (font (size 1 1) (thickness 0.15)))
+    )
+    (fp_line (start -1.15 -0.6) (end 1.15 -0.6) (layer F.CrtYd) (width 0.05))
+    (fp_line (start -1.15 0.6) (end 1.15 0.6) (layer F.CrtYd) (width 0.05))
+    (fp_line (start -1.15 -0.6) (end -1.15 0.6) (layer F.CrtYd) (width 0.05))
+    (fp_line (start 1.15 -0.6) (end 1.15 0.6) (layer F.CrtYd) (width 0.05))
+    (fp_line (start 0.25 -0.475) (end -0.25 -0.475) (layer F.SilkS) (width 0.15))
+    (fp_line (start -0.25 0.475) (end 0.25 0.475) (layer F.SilkS) (width 0.15))
+    (pad 1 smd rect (at -0.55 0) (size 0.6 0.5) (layers F.Cu F.Paste F.Mask)
+      (net 8 +3V3))
+    (pad 2 smd rect (at 0.55 0) (size 0.6 0.5) (layers F.Cu F.Paste F.Mask)
+      (net 6 GND))
+    (model Capacitors_SMD.3dshapes/C_0402.wrl
+      (at (xyz 0 0 0))
+      (scale (xyz 1 1 1))
+      (rotate (xyz 0 0 0))
+    )
+  )
+  (module Capacitors_SMD:C_0402 (layer F.Cu)
+    (at 22.86 37.719)
+    (descr "Capacitor SMD 0402, reflow soldering, AVX (see smccp.pdf)")
+    (tags "capacitor 0402")
+    (attr smd)
+    (fp_text reference C10 (at 0 -1.7) (layer F.SilkS)
+      (effects (font (size 1 1) (thickness 0.15)))
+    )
+    (fp_text value 0.1uF (at 0 1.7) (layer F.Fab)
+      (effects (font (size 1 1) (thickness 0.15)))
+    )
+    (fp_line (start -1.15 -0.6) (end 1.15 -0.6) (layer F.CrtYd) (width 0.05))
+    (fp_line (start -1.15 0.6) (end 1.15 0.6) (layer F.CrtYd) (width 0.05))
+    (fp_line (start -1.15 -0.6) (end -1.15 0.6) (layer F.CrtYd) (width 0.05))
+    (fp_line (start 1.15 -0.6) (end 1.15 0.6) (layer F.CrtYd) (width 0.05))
+    (fp_line (start 0.25 -0.475) (end -0.25 -0.475) (layer F.SilkS) (width 0.15))
+    (fp_line (start -0.25 0.475) (end 0.25 0.475) (layer F.SilkS) (width 0.15))
+    (pad 1 smd rect (at -0.55 0) (size 0.6 0.5) (layers F.Cu F.Paste F.Mask)
+      (net 8 +3V3))
+    (pad 2 smd rect (at 0.55 0) (size 0.6 0.5) (layers F.Cu F.Paste F.Mask)
+      (net 6 GND))
+    (model Capacitors_SMD.3dshapes/C_0402.wrl
+      (at (xyz 0 0 0))
+      (scale (xyz 1 1 1))
+      (rotate (xyz 0 0 0))
+    )
+  )
+  (module SMD:R-PWSON-N10 (layer F.Cu)
+    (at 26.924 30.734)
+    (fp_text reference U1 (at 0 1.905) (layer F.SilkS)
+      (effects (font (size 1 1) (thickness 0.15)))
+    )
+    (fp_text value bq24040 (at 0 -2.032) (layer F.Fab)
+      (effects (font (size 1 1) (thickness 0.15)))
+    )
+    (fp_circle (center -1.27 -1.397) (end -1.016 -1.524) (layer F.SilkS) (width 0.15))
+    (pad 1 smd rect (at -1.2 -0.8) (size 1 0.23) (layers F.Cu F.Paste F.Mask))
+    (pad 2 smd rect (at -1.2 -0.4) (size 1 0.23) (layers F.Cu F.Paste F.Mask))
+    (pad 3 smd rect (at -1.2 0) (size 1 0.23) (layers F.Cu F.Paste F.Mask))
+    (pad 4 smd rect (at -1.2 0.4) (size 1 0.23) (layers F.Cu F.Paste F.Mask))
+    (pad 5 smd rect (at -1.2 0.8) (size 1 0.23) (layers F.Cu F.Paste F.Mask))
+    (pad 6 smd rect (at 1.2 0.8) (size 1 0.23) (layers F.Cu F.Paste F.Mask))
+    (pad 7 smd rect (at 1.2 0.4) (size 1 0.23) (layers F.Cu F.Paste F.Mask))
+    (pad 8 smd rect (at 1.2 0) (size 1 0.23) (layers F.Cu F.Paste F.Mask))
+    (pad 9 smd rect (at 1.2 -0.4) (size 1 0.23) (layers F.Cu F.Paste F.Mask))
+    (pad 10 smd rect (at 1.2 -0.8) (size 1 0.23) (layers F.Cu F.Paste F.Mask)
+      (net 10 /VOUT))
+    (pad PAD smd rect (at 0 0) (size 0.7 1.2) (layers F.Cu F.Paste F.Mask))
+  )
+  (module TO_SOT_Packages_SMD:SOT-23-5 (layer F.Cu)
+    (at 29.083 41.91)
+    (descr "5-pin SOT23 package")
+    (tags SOT-23-5)
+    (attr smd)
+    (fp_text reference U2 (at -0.05 -2.55) (layer F.SilkS)
+      (effects (font (size 1 1) (thickness 0.15)))
+    )
+    (fp_text value tps62200 (at -0.05 2.35) (layer F.Fab)
+      (effects (font (size 1 1) (thickness 0.15)))
+    )
+    (fp_line (start -1.8 -1.6) (end 1.8 -1.6) (layer F.CrtYd) (width 0.05))
+    (fp_line (start 1.8 -1.6) (end 1.8 1.6) (layer F.CrtYd) (width 0.05))
+    (fp_line (start 1.8 1.6) (end -1.8 1.6) (layer F.CrtYd) (width 0.05))
+    (fp_line (start -1.8 1.6) (end -1.8 -1.6) (layer F.CrtYd) (width 0.05))
+    (fp_circle (center -0.3 -1.7) (end -0.2 -1.7) (layer F.SilkS) (width 0.15))
+    (fp_line (start 0.25 -1.45) (end -0.25 -1.45) (layer F.SilkS) (width 0.15))
+    (fp_line (start 0.25 1.45) (end 0.25 -1.45) (layer F.SilkS) (width 0.15))
+    (fp_line (start -0.25 1.45) (end 0.25 1.45) (layer F.SilkS) (width 0.15))
+    (fp_line (start -0.25 -1.45) (end -0.25 1.45) (layer F.SilkS) (width 0.15))
+    (pad 1 smd rect (at -1.1 -0.95) (size 1.06 0.65) (layers F.Cu F.Paste F.Mask)
+      (net 10 /VOUT))
+    (pad 2 smd rect (at -1.1 0) (size 1.06 0.65) (layers F.Cu F.Paste F.Mask)
+      (net 6 GND))
+    (pad 3 smd rect (at -1.1 0.95) (size 1.06 0.65) (layers F.Cu F.Paste F.Mask)
+      (net 10 /VOUT))
+    (pad 4 smd rect (at 1.1 0.95) (size 1.06 0.65) (layers F.Cu F.Paste F.Mask)
+      (net 8 +3V3))
+    (pad 5 smd rect (at 1.1 -0.95) (size 1.06 0.65) (layers F.Cu F.Paste F.Mask))
+    (model TO_SOT_Packages_SMD.3dshapes/SOT-23-5.wrl
+      (at (xyz 0 0 0))
+      (scale (xyz 1 1 1))
+      (rotate (xyz 0 0 0))
+    )
