File: pcb/cubecast.sch (KiCad schematic (older format))
At the start: 15 parts, among them U1 bq24040, U2 tps62200

Commit message: PCB started
Parts:
- OLED1: footprint (none) -> OLED:OLED_0.66_inch_64x48
- gave numbers to parts that had none: 7
Changed lines of the file:
@@
 F 0 "OLED1" H 8500 2150 60  0000 C CNB
 F 1 "OLED_0.66_inch_64x48" V 8800 600 60  0000 C CNB
-F 2 "" H 8750 1900 60  0000 C CNN
+F 2 "OLED:OLED_0.66_inch_64x48" H 8750 1900 60  0001 C CNN
 F 3 "" H 8750 1900 60  0000 C CNN
 	1    8800 1950
@@
 	9600 3800 9600 3700
 $Comp
-L GND #PWR2
+L GND #PWR7
 U 1 1 55C688E0
 P 9600 4450
-F 0 "#PWR2" H 9600 4200 50  0001 C CNN
+F 0 "#PWR7" H 9600 4200 50  0001 C CNN
 F 1 "GND" H 9600 4300 50  0000 C CNN
 F 2 "" H 9600 4450 60  0000 C CNN
@@
 Connection ~ 9600 4150
 $Comp
-L +3.3V #PWR1
+L +3.3V #PWR6
 U 1 1 55C6898E
 P 9600 1850
-F 0 "#PWR1" H 9600 1700 50  0001 C CNN
+F 0 "#PWR6" H 9600 1700 50  0001 C CNN
 F 1 "+3.3V" H 9600 1990 50  0000 C CNN
 F 2 "" H 9600 1850 60  0000 C CNN
@@
 $EndComp
 $Comp
-L GND #PWR3
+L GND #PWR8
 U 1 1 55C68BAC
 P 10400 2750
-F 0 "#PWR3" H 10400 2500 50  0001 C CNN
+F 0 "#PWR8" H 10400 2500 50  0001 C CNN
 F 1 "GND" H 10400 2600 50  0000 C CNN
 F 2 "" H 10400 2750 60  0000 C CNN
@@
 $EndComp
 $Comp
-L +3.3V #PWR?
+L +3.3V #PWR4
 U 1 1 55C693B9
 P 7100 1650
-F 0 "#PWR?" H 7100 1500 50  0001 C CNN
+F 0 "#PWR4" H 7100 1500 50  0001 C CNN
 F 1 "+3.3V" H 7100 1790 50  0000 C CNN
 F 2 "" H 7100 1650 60  0000 C CNN
@@
 $EndComp
 $Comp
-L INDUCTOR_SMALL L?
+L INDUCTOR_SMALL L1
 U 1 1 55C693E5
 P 6800 1800
-F 0 "L?" H 6800 1900 50  0000 C CNN
+F 0 "L1" H 6800 1900 50  0000 C CNN
 F 1 "10uH" H 6800 1750 50  0000 C CNN
 F 2 "" H 6800 1800 60  0000 C CNN
@@
 $EndComp
 $Comp
-L C_Small C?
+L C_Small C6
 U 1 1 55C694BC
 P 7100 2000
-F 0 "C?" H 7110 2070 50  0000 L CNN
+F 0 "C6" H 7110 2070 50  0000 L CNN
 F 1 "10uF" H 7110 1920 50  0000 L CNN
 F 2 "Capacitors_SMD:C_0603_HandSoldering" H 7100 2000 60  0001 C CNN
@@
 Connection ~ 4700 1800
 $Comp
-L CONN_01X01 P?
+L CONN_01X01 P1
 U 1 1 55C699CD
 P 4700 1400
-F 0 "P?" H 4700 1500 50  0000 C CNN
+F 0 "P1" H 4700 1500 50  0000 C CNN
 F 1 "TP" V 4800 1400 50  0000 C CNN
 F 2 "" H 4700 1400 60  0000 C CNN
@@
 VOUT
 $Comp
-L GND #PWR?
+L GND #PWR3
 U 1 1 55C69B22
 P 5250 2150
-F 0 "#PWR?" H 5250 1900 50  0001 C CNN
+F 0 "#PWR3" H 5250 1900 50  0001 C CNN
 F 1 "GND" H 5250 2000 50  0000 C CNN
 F 2 "" H 5250 2150 60  0000 C CNN
@@
 $EndComp
 $Comp
-L C_Small C?
+L C_Small C5
 U 1 1 55C69C7F
 P 5250 1900
-F 0 "C?" H 5260 1970 50  0000 L CNN
+F 0 "C5" H 5260 1970 50  0000 L CNN
 F 1 "10uF" H 5260 1820 50  0000 L CNN
 F 2 "Capacitors_SMD:C_0603_HandSoldering" H 5250 1900 60  0001 C CNN
@@
 	5250 2000 5250 2150
 $Comp
-L ESP-07v2 U?
+L ESP-07v2 U3
 U 1 1 55C68E66
 P 3400 4450
-F 0 "U?" H 3950 5100 50  0000 C CNN
+F 0 "U3" H 3950 5100 50  0000 C CNN
 F 1 "ESP-07v2" H 3400 4550 50  0000 C CNN
 F 2 "ESP8266:ESP-07v2" H 3400 4450 50  0001 C CNN
@@
 $EndComp
 $Comp
-L C_Small C?
+L C_Small C8
 U 1 1 55C6921F
 P 10950 1850
-F 0 "C?" H 10960 1920 50  0000 L CNN
+F 0 "C8" H 10960 1920 50  0000 L CNN
 F 1 "0.1uF" H 10960 1770 50  0000 L CNN
 F 2 "Capacitors_SMD:C_0402" H 10950 1850 60  0001 C CNN
@@
 $EndComp
 $Comp
-L C_Small C?
+L C_Small C7
 U 1 1 55C69387
 P 10650 1850
-F 0 "C?" H 10660 1920 50  0000 L CNN
+F 0 "C7" H 10660 1920 50  0000 L CNN
 F 1 "0.1uF" H 10660 1770 50  0000 L CNN
 F 2 "Capacitors_SMD:C_0402" H 10650 1850 60  0001 C CNN
@@
 	10650 1700 10650 1750
 $Comp
-L +3.3V #PWR?
+L +3.3V #PWR9
 U 1 1 55C695D0
 P 10950 1650
-F 0 "#PWR?" H 10950 1500 50  0001 C CNN
+F 0 "#PWR9" H 10950 1500 50  0001 C CNN
 F 1 "+3.3V" H 10950 1790 50  0000 C CNN
 F 2 "" H 10950 1650 60  0000 C CNN
@@
 $EndComp
 $Comp
-L GND #PWR?
+L GND #PWR10
 U 1 1 55C69602
 P 10950 2050
-F 0 "#PWR?" H 10950 1800 50  0001 C CNN
+F 0 "#PWR10" H 10950 1800 50  0001 C CNN
 F 1 "GND" H 10950 1900 50  0000 C CNN
 F 2 "" H 10950 2050 60  0000 C CNN
@@
 Connection ~ 10950 2000
 $Comp
-L GND #PWR?
+L GND #PWR5
 U 1 1 55C698DC
 P 7100 2200
-F 0 "#PWR?" H 7100 1950 50  0001 C CNN
+F 0 "#PWR5" H 7100 1950 50  0001 C CNN
 F 1 "GND" H 7100 2050 50  0000 C CNN
 F 2 "" H 7100 2200 60  0000 C CNN
@@
 $EndComp
 $Comp
-L GND #PWR?
+L GND #PWR2
 U 1 1 55C69977
 P 3400 5450
-F 0 "#PWR?" H 3400 5200 50  0001 C CNN
+F 0 "#PWR2" H 3400 5200 50  0001 C CNN
 F 1 "GND" H 3400 5300 50  0000 C CNN
 F 2 "" H 3400 5450 60  0000 C CNN
@@
 $EndComp
 $Comp
-L +3.3V #PWR?
+L +3.3V #PWR1
 U 1 1 55C69A0F
 P 3400 3450
-F 0 "#PWR?" H 3400 3300 50  0001 C CNN
+F 0 "#PWR1" H 3400 3300 50  0001 C CNN
 F 1 "+3.3V" H 3400 3590 50  0000 C CNN
 F 2 "" H 3400 3450 60  0000 C CNN

Commit message: initial placement
Parts:
- added C10, C9: 0.1uF, Capacitors_SMD:C_0402, symbol C_Small
Connections:
- net +3V3: now also C10.1, C9.1
- net GND: now also U3.9 (GND), C10.2, C9.2
Changed lines of the file:
@@
 	9600 3800 9600 3700
 $Comp
-L GND #PWR7
+L GND #PWR9
 U 1 1 55C688E0
 P 9600 4450
-F 0 "#PWR7" H 9600 4200 50  0001 C CNN
+F 0 "#PWR9" H 9600 4200 50  0001 C CNN
 F 1 "GND" H 9600 4300 50  0000 C CNN
 F 2 "" H 9600 4450 60  0000 C CNN
@@
 Connection ~ 9600 4150
 $Comp
-L +3.3V #PWR6
+L +3.3V #PWR8
 U 1 1 55C6898E
 P 9600 1850
-F 0 "#PWR6" H 9600 1700 50  0001 C CNN
+F 0 "#PWR8" H 9600 1700 50  0001 C CNN
 F 1 "+3.3V" H 9600 1990 50  0000 C CNN
 F 2 "" H 9600 1850 60  0000 C CNN
@@
 $EndComp
 $Comp
-L GND #PWR8
+L GND #PWR10
 U 1 1 55C68BAC
 P 10400 2750
-F 0 "#PWR8" H 10400 2500 50  0001 C CNN
+F 0 "#PWR10" H 10400 2500 50  0001 C CNN
 F 1 "GND" H 10400 2600 50  0000 C CNN
 F 2 "" H 10400 2750 60  0000 C CNN
@@
 $EndComp
 $Comp
-L +3.3V #PWR4
+L +3.3V #PWR6
 U 1 1 55C693B9
 P 7100 1650
-F 0 "#PWR4" H 7100 1500 50  0001 C CNN
+F 0 "#PWR6" H 7100 1500 50  0001 C CNN
 F 1 "+3.3V" H 7100 1790 50  0000 C CNN
 F 2 "" H 7100 1650 60  0000 C CNN
@@
 VOUT
 $Comp
-L GND #PWR3
+L GND #PWR5
 U 1 1 55C69B22
 P 5250 2150
-F 0 "#PWR3" H 5250 1900 50  0001 C CNN
+F 0 "#PWR5" H 5250 1900 50  0001 C CNN
 F 1 "GND" H 5250 2000 50  0000 C CNN
 F 2 "" H 5250 2150 60  0000 C CNN
@@
 	10650 1700 10650 1750
 $Comp
-L +3.3V #PWR9
+L +3.3V #PWR11
 U 1 1 55C695D0
 P 10950 1650
-F 0 "#PWR9" H 10950 1500 50  0001 C CNN
+F 0 "#PWR11" H 10950 1500 50  0001 C CNN
 F 1 "+3.3V" H 10950 1790 50  0000 C CNN
 F 2 "" H 10950 1650 60  0000 C CNN
@@
 $EndComp
 $Comp
-L GND #PWR10
+L GND #PWR12
 U 1 1 55C69602
 P 10950 2050
-F 0 "#PWR10" H 10950 1800 50  0001 C CNN
+F 0 "#PWR12" H 10950 1800 50  0001 C CNN
 F 1 "GND" H 10950 1900 50  0000 C CNN
 F 2 "" H 10950 2050 60  0000 C CNN
@@
 Connection ~ 10950 2000
 $Comp
-L GND #PWR5
+L GND #PWR7
 U 1 1 55C698DC
 P 7100 2200
-F 0 "#PWR5" H 7100 1950 50  0001 C CNN
+F 0 "#PWR7" H 7100 1950 50  0001 C CNN
 F 1 "GND" H 7100 2050 50  0000 C CNN
 F 2 "" H 7100 2200 60  0000 C CNN
@@
 Wire Wire Line
 	3400 3450 3400 3550
+$Comp
+L C_Small C9
+U 1 1 55C89A4F
+P 5150 4350
+F 0 "C9" H 5160 4420 50  0000 L CNN
+F 1 "0.1uF" H 5160 4270 50  0000 L CNN
+F 2 "Capacitors_SMD:C_0402" H 5150 4350 60  0001 C CNN
+F 3 "" H 5150 4350 60  0000 C CNN
+	1    5150 4350
+	1    0    0    -1
+$EndComp
+$Comp
+L C_Small C10
+U 1 1 55C89AB2
+P 5450 4350
+F 0 "C10" H 5460 4420 50  0000 L CNN
+F 1 "0.1uF" H 5460 4270 50  0000 L CNN
+F 2 "Capacitors_SMD:C_0402" H 5450 4350 60  0001 C CNN
+F 3 "" H 5450 4350 60  0000 C CNN
+	1    5450 4350
+	1    0    0    -1
+$EndComp
+Wire Wire Line
+	3400 5350 3400 5450
+Wire Wire Line
+	5150 4050 5150 4250
+Wire Wire Line
+	5150 4150 5450 4150
+Wire Wire Line
+	5450 4150 5450 4250
+Wire Wire Line
+	5450 4450 5450 4550
+Wire Wire Line
+	5450 4550 5150 4550
+Wire Wire Line
+	5150 4450 5150 4600
+$Comp
+L GND #PWR4
+U 1 1 55C89CB3
+P 5150 4600
+F 0 "#PWR4" H 5150 4350 50  0001 C CNN
+F 1 "GND" H 5150 4450 50  0000 C CNN
+F 2 "" H 5150 4600 60  0000 C CNN
+F 3 "" H 5150 4600 60  0000 C CNN
+	1    5150 4600
+	1    0    0    -1
+$EndComp
+$Comp
+L +3V3 #PWR3
+U 1 1 55C89D60
+P 5150 4050
+F 0 "#PWR3" H 5150 3900 50  0001 C CNN
+F 1 "+3V3" H 5150 4190 50  0000 C CNN
+F 2 "" H 5150 4050 60  0000 C CNN
+F 3 "" H 5150 4050 60  0000 C CNN
+	1    5150 4050
+	1    0    0    -1
+$EndComp
+Connection ~ 5150 4150
+Connection ~ 5150 4550
 $EndSCHEMATC

Commit message: footprint for charger
Parts:
- U1: footprint (none) -> SMD:R-PWSON-N10
- U2: footprint (none) -> TO_SOT_Packages_SMD:SOT-23-5
Other:
- moved on the sheet: C5, C6, L1, P1, U1, U2
Changed lines of the file:
@@
 L bq24040 U1
 U 1 1 55C68F96
-P 3550 2450
-F 0 "U1" H 3250 3250 60  0000 C CNB
-F 1 "bq24040" H 3800 2450 60  0000 C CNB
-F 2 "" H 3550 2450 60  0000 C CNN
-F 3 "" H 3550 2450 60  0000 C CNN
-	1    3550 2450
+P 1900 2350
+F 0 "U1" H 1600 3150 60  0000 C CNB
+F 1 "bq24040" H 2150 2350 60  0000 C CNB
+F 2 "SMD:R-PWSON-N10" H 1900 2350 60  0001 C CNN
+F 3 "" H 1900 2350 60  0000 C CNN
+	1    1900 2350
 	1    0    0    -1
 $EndComp
@@
 L tps62200 U2
 U 1 1 55C6910F
-P 6000 1900
-F 0 "U2" H 5750 2150 60  0000 C CNB
-F 1 "tps62200" H 6000 1650 60  0000 C CNN
-F 2 "" H 6000 1900 60  0000 C CNN
-F 3 "" H 6000 1900 60  0000 C CNN
-	1    6000 1900
+P 4350 1800
+F 0 "U2" H 4100 2050 60  0000 C CNB
+F 1 "tps62200" H 4350 1550 60  0000 C CNN
+F 2 "TO_SOT_Packages_SMD:SOT-23-5" H 4350 1800 60  0001 C CNN
+F 3 "" H 4350 1800 60  0000 C CNN
+	1    4350 1800
 	1    0    0    -1
 $EndComp
@@
 L +3.3V #PWR6
 U 1 1 55C693B9
-P 7100 1650
-F 0 "#PWR6" H 7100 1500 50  0001 C CNN
-F 1 "+3.3V" H 7100 1790 50  0000 C CNN
-F 2 "" H 7100 1650 60  0000 C CNN
-F 3 "" H 7100 1650 60  0000 C CNN
-	1    7100 1650
+P 5450 1550
+F 0 "#PWR6" H 5450 1400 50  0001 C CNN
+F 1 "+3.3V" H 5450 1690 50  0000 C CNN
+F 2 "" H 5450 1550 60  0000 C CNN
+F 3 "" H 5450 1550 60  0000 C CNN
+	1    5450 1550
 	1    0    0    -1
 $EndComp
@@
 L INDUCTOR_SMALL L1
 U 1 1 55C693E5
-P 6800 1800
-F 0 "L1" H 6800 1900 50  0000 C CNN
-F 1 "10uH" H 6800 1750 50  0000 C CNN
-F 2 "" H 6800 1800 60  0000 C CNN
-F 3 "" H 6800 1800 60  0000 C CNN
-	1    6800 1800
+P 5150 1700
+F 0 "L1" H 5150 1800 50  0000 C CNN
+F 1 "10uH" H 5150 1650 50  0000 C CNN
+F 2 "" H 5150 1700 60  0000 C CNN
+F 3 "" H 5150 1700 60  0000 C CNN
+	1    5150 1700
 	1    0    0    -1
 $EndComp
@@
 L C_Small C6
 U 1 1 55C694BC
-P 7100 2000
-F 0 "C6" H 7110 2070 50  0000 L CNN
-F 1 "10uF" H 7110 1920 50  0000 L CNN
-F 2 "Capacitors_SMD:C_0603_HandSoldering" H 7100 2000 60  0001 C CNN
-F 3 "" H 7100 2000 60  0000 C CNN
-	1    7100 2000
+P 5450 1900
+F 0 "C6" H 5460 1970 50  0000 L CNN
+F 1 "10uF" H 5460 1820 50  0000 L CNN
+F 2 "Capacitors_SMD:C_0603_HandSoldering" H 5450 1900 60  0001 C CNN
+F 3 "" H 5450 1900 60  0000 C CNN
+	1    5450 1900
 	1    0    0    -1
 $EndComp
 Wire Wire Line
-	6450 1800 6550 1800
+	4800 1700 4900 1700
 Wire Wire Line
-	7050 1800 7100 1800
+	5400 1700 5450 1700
 Wire Wire Line
-	7100 1650 7100 1900
-Connection ~ 7100 1800
+	5450 1550 5450 1800
+Connection ~ 5450 1700
 Wire Wire Line
-	7100 2100 7100 2200
+	5450 2000 5450 2100
 Wire Wire Line
-	6450 2000 6950 2000
+	4800 1900 5300 1900
 Wire Wire Line
-	6950 2000 7100 1800
+	5300 1900 5450 1700
 Wire Wire Line
-	5500 1900 5450 1900
+	3850 1800 3800 1800
 Wire Wire Line
-	5450 1900 5450 1800
-Connection ~ 5450 1800
+	3800 1800 3800 1700
+Connection ~ 3800 1700
 Wire Wire Line
-	4700 1600 4700 1800
-Connection ~ 4700 1800
+	3050 1500 3050 1700
+Connection ~ 3050 1700
 $Comp
 L CONN_01X01 P1
 U 1 1 55C699CD
-P 4700 1400
-F 0 "P1" H 4700 1500 50  0000 C CNN
-F 1 "TP" V 4800 1400 50  0000 C CNN
-F 2 "" H 4700 1400 60  0000 C CNN
-F 3 "" H 4700 1400 60  0000 C CNN
-	1    4700 1400
+P 3050 1300
+F 0 "P1" H 3050 1400 50  0000 C CNN
+F 1 "TP" V 3150 1300 50  0000 C CNN
+F 2 "" H 3050 1300 60  0000 C CNN
+F 3 "" H 3050 1300 60  0000 C CNN
+	1    3050 1300
 	0    -1   -1   0
 $EndComp
-Text Label 4250 1800 0    60   ~ 0
+Text Label 2600 1700 0    60   ~ 0
 VOUT
 $Comp
 L GND #PWR5
 U 1 1 55C69B22
-P 5250 2150
-F 0 "#PWR5" H 5250 1900 50  0001 C CNN
-F 1 "GND" H 5250 2000 50  0000 C CNN
-F 2 "" H 5250 2150 60  0000 C CNN
-F 3 "" H 5250 2150 60  0000 C CNN
-	1    5250 2150
+P 3600 2050
+F 0 "#PWR5" H 3600 1800 50  0001 C CNN
+F 1 "GND" H 3600 1900 50  0000 C CNN
+F 2 "" H 3600 2050 60  0000 C CNN
+F 3 "" H 3600 2050 60  0000 C CNN
+	1    3600 2050
 	1    0    0    -1
 $EndComp
@@
 L C_Small C5
 U 1 1 55C69C7F
-P 5250 1900
-F 0 "C5" H 5260 1970 50  0000 L CNN
-F 1 "10uF" H 5260 1820 50  0000 L CNN
-F 2 "Capacitors_SMD:C_0603_HandSoldering" H 5250 1900 60  0001 C CNN
-F 3 "" H 5250 1900 60  0000 C CNN
-	1    5250 1900
+P 3600 1800
+F 0 "C5" H 3610 1870 50  0000 L CNN
+F 1 "10uF" H 3610 1720 50  0000 L CNN
+F 2 "Capacitors_SMD:C_0603_HandSoldering" H 3600 1800 60  0001 C CNN
+F 3 "" H 3600 1800 60  0000 C CNN
+	1    3600 1800
 	1    0    0    -1
 $EndComp
 Wire Wire Line
-	4200 1800 5500 1800
-Connection ~ 5250 1800
+	2550 1700 3850 1700
+Connection ~ 3600 1700
 Wire Wire Line
-	5500 2000 5250 2000
+	3850 1900 3600 1900
 Wire Wire Line
-	5250 2000 5250 2150
+	3600 1900 3600 2050
 $Comp
 L ESP-07v2 U3
@@
 L GND #PWR7
 U 1 1 55C698DC
-P 7100 2200
-F 0 "#PWR7" H 7100 1950 50  0001 C CNN
-F 1 "GND" H 7100 2050 50  0000 C CNN
-F 2 "" H 7100 2200 60  0000 C CNN
-F 3 "" H 7100 2200 60  0000 C CNN
-	1    7100 2200
+P 5450 2100
+F 0 "#PWR7" H 5450 1850 50  0001 C CNN
+F 1 "GND" H 5450 1950 50  0000 C CNN
+F 2 "" H 5450 2100 60  0000 C CNN
+F 3 "" H 5450 2100 60  0000 C CNN
+	1    5450 2100
 	1    0    0    -1
 $EndComp
